Commit message: launch

File: eu_map_Exported/eu_map/eu_map.urdf (robot description, URDF)
Before this commit: robot eu_map, 5 links, 4 joints
Links:
- link base: geometry collision mesh filename=package://Eurodot_2018_gazebo/eu_map_Exported/eu_map/collis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; visual mesh filename=package://Eurodot_2018_gazebo/eu_map_Exported/eu_map/visual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
- link green: geometry collision mesh filename=package://Eurodot_2018_gazebo/eu_map_Exported/eu_map/collis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; visual mesh filename=package://Eurodot_2018_gazebo/eu_map_Exported/eu_map/visual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
- link rad: geometry collision mesh filename=package://Eurodot_2018_gazebo/eu_map_Exported/eu_map/collis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; visual mesh filename=package://Eurodot_2018_gazebo/eu_map_Exported/eu_map/visual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
- link wall: geometry collision mesh filename=package://Eurodot_2018_gazebo/eu_map_Exported/eu_map/collis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; visual mesh filename=package://Eurodot_2018_gazebo/eu_map_Exported/eu_map/visual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
- link wall2: geometry collision mesh filename=package://Eurodot_2018_gazebo/eu_map_Exported/eu_map/collis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; visual mesh filename=package://Eurodot_2018_gazebo/eu_map_Exported/eu_map/visual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

Commit message: fix

File: eu_map_Exported/eu_map/eu_map.urdf (robot description, URDF)
Before this commit: robot eu_map, 5 links, 4 joints
Links:
- link base: geometry collision mesh filename=package://Eurodot2018_gazebo/eu_map_Exported/eu_map/collisi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; visual mesh filename=package://Eurodot2018_gazebo/eu_map_Exported/eu_map/visualS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
- link green: geometry collision mesh filename=package://Eurodot2018_gazebo/eu_map_Exported/eu_map/collisi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; visual mesh filename=package://Eurodot2018_gazebo/eu_map_Exported/eu_map/visualS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
- link rad: geometry collision mesh filename=package://Eurodot2018_gazebo/eu_map_Exported/eu_map/collisi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; visual mesh filename=package://Eurodot2018_gazebo/eu_map_Exported/eu_map/visualS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
- link wall: geometry collision mesh filename=package://Eurodot2018_gazebo/eu_map_Exported/eu_map/collisi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; visual mesh filename=package://Eurodot2018_gazebo/eu_map_Exported/eu_map/visualS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
- link wall2: geometry collision mesh filename=package://Eurodot2018_gazebo/eu_map_Exported/eu_map/collisi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; visual mesh filename=package://Eurodot2018_gazebo/eu_map_Exported/eu_map/visualS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
