Commit message: car test 2

File: TEST/assam/robots/assam.urdf (robot description, URDF)
Before this commit: robot assam, 4 links, 3 joints
Joints:
- joint j2: limit effort=0 velocity=0 -> (none); type revolute -> continuous
- joint j3: origin xyz=0.00358608863369358 -0.41 -6.86334715221801E-05 rpy=-6.12303176911189E-17 0 0 -> xyz=0.0035861 -0.41 -6.8633E-05 rpy=-6.123E-17 0 0; type revolute -> continuous

Commit message: car test 3

File: TEST/assam/robots/assam.urdf (robot description, URDF)
Before this commit: robot assam, 4 links, 3 joints
Links:
- link base_link: mass 1.68994026795429 -> 5
- link w1: mass 0.098005596771295 -> 1
- link w2: mass 0.098005596771295 -> 1
- link w3: mass 0.098005596771295 -> 1
Joints:
- joint j1: axis 1 0 0 -> 0 -1 0; origin xyz=0.0035861 -0.41 -6.8633E-05 rpy=-6.123E-17 0 0 -> xyz=0.21 0 -0.015 rpy=0 0 0
- joint j2: axis 1 0 0 -> 0 -1 0; origin xyz=0.0035861 -0.41 -6.8633E-05 rpy=-6.123E-17 0 0 -> xyz=0 0.115 -0.015 rpy=0 0 0
- joint j3: axis 1 0 0 -> 0 -1 0; origin xyz=0.0035861 -0.41 -6.8633E-05 rpy=-6.123E-17 0 0 -> xyz=0 -0.115 -0.015 rpy=0 0 0

Commit message: car test 4

File: TEST/assam/robots/assam.urdf (robot description, URDF)
Before this commit: robot assam, 4 links, 3 joints
Links:
- link base_link: mass 5 -> 1.6899
- link w1: mass 1 -> 0.09722
- link w2: mass 1 -> 0.09722
- link w3: mass 1 -> 0.09722
