Commit message: test2-2

File: test2/minicar2/robots/minicar2.urdf (robot description, URDF)
Before this commit: robot minicar, 3 links, 2 joints
Links:
- removed link l_wh
- removed link r_wl
- added link wl, mass 1; collision mesh filename=package://minicar2/meshes/wl.STL; visual mesh filename=package://minicar2/meshes/wl.STL
- added link wr, mass 1; collision mesh filename=package://minicar2/meshes/wr.STL; visual mesh filename=package://minicar2/meshes/wr.STL
- link base_link: mass 0.60636 -> 5; geometry collision mesh filename=package://minicar2/meshes/base_link.STL; visual mesh filename=package://minicar2/meshes/base_link.STL
Joints:
- removed joint j1
- removed joint j2
- added joint jl: type continuous, parent base_link, child wl, origin xyz=0 0.06 -0.015 rpy=0 0 0, axis 0 1 0
- added joint jr: type continuous, parent base_link, child wr, origin xyz=0 -0.06 -0.015 rpy=0 0 0, axis 0 0.99083 0.13511
